Commit message: Update description

File: urdf/common/gazebo.urdf.xacro (robot description, xacro)
@@ -7,6 +7,6 @@
         <parameters>${config_file}</parameters>
         <ros>
-          <namespace>${namespace}</namespace>
-          <remapping>drive_controller/cmd_vel:=cmd_vel</remapping>
+          <namespace>$(arg namespace)</namespace>
+          <remapping>drive_controller/cmd_vel_unstamped:=cmd_vel</remapping>
           <remapping>drive_controller/odom:=odometry/wheels</remapping>
           <remapping>drive_controller/transition_event:=drive_controller/_transition_event</remapping>

File: urdf/common/wheel.urdf.xacro (robot description, xacro)
@@ -73,21 +73,4 @@
       </inertial>
     </link>
-    <xacro:if value="${use_sim}">
-      <xacro:if value="${config['mecanum']}">
-        <gazebo reference="${prefix}_wheel_link" xmlns:ignition="http://ignitionrobotics.org/schema">
-          <collision>
-            <surface>
-              <friction>
-                <ode>
-                  <mu>1.0</mu>
-                  <mu2>0.0</mu2>
-                  <fdir1 ignition:expressed_in="base_link">${fdir}</fdir1>
-                </ode>
-              </friction>
-            </surface>
-          </collision>
-        </gazebo>
-      </xacro:if>
-    </xacro:if>
   </xacro:macro>
 </robot>

File: urdf/rover_a1.urdf.xacro (robot description, xacro)
@@ -1,5 +1,5 @@
 <?xml version="1.0" encoding="utf-8"?>
 <robot name="rover_a1" xmlns:xacro="http://wiki.ros.org/xacro">
-  <xacro:arg name="use_sim" default="true" />
+  <xacro:arg name="use_sim" default="false" />
   <xacro:arg name="wheel_config_file"
     default="$(find rover_description)/config/wheel_01.yaml" />

File: urdf/rover_a1/rover_a1_macro.urdf.xacro (robot description, xacro)
@@ -5,5 +5,5 @@
     params="wheel_config_file
             controller_config_file
-            use_sim:=true
+            use_sim:=false
             namespace:=''">
     <xacro:property name="ns" value='${namespace + "/" if namespace else ""}' />
@@ -11,12 +11,9 @@
     <xacro:property name="wheelbase" value="0.2542" />
     <xacro:property name="wheel_mount_point_y" value="0.31301" />
-    <!-- INCLUDE ROBOT PARTS DEFINITIONS -->
     <xacro:include filename="$(find rover_description)/urdf/rover_a1/base.urdf.xacro" ns="body" />
+    <xacro:include filename="$(find rover_description)/urdf/common/wheel.urdf.xacro" ns="wheel" />
     <xacro:include filename="$(find rover_description)/urdf/common/gazebo.urdf.xacro" ns="gazebo" />
-    <xacro:include filename="$(find rover_description)/urdf/common/wheel.urdf.xacro" ns="wheel" />
-    <!-- BODY DECLARATION -->
     <xacro:body.body
       wheel_radius="${wheel_config['wheel_radius']}" />
-    <!-- WHEEL DECLARATION -->
     <xacro:wheel.wheel
       config="${wheel_config}"
@@ -39,4 +36,39 @@
       mount_point_y="${wheel_mount_point_y}"
       prefix="rr" />
+    <!-- ROS2 Controller -->
+    <ros2_control name="${ns}rover_system" type="system">
+      <!-- Gazebo simulation system contorller -->
+      <hardware>
+        <plugin>gz_ros2_control/GazeboSimSystem</plugin>
+      </hardware>
+      <joint name="fl_wheel_base_to_fl_wheel_joint">
+        <command_interface name="velocity" />
+        <state_interface name="position" />
+        <state_interface name="velocity" />
+        <state_interface name="effort" />
+      </joint>
+      <joint name="fr_wheel_base_to_fr_wheel_joint">
+        <command_interface name="velocity" />
+        <state_interface name="position" />
+        <state_interface name="velocity" />
+        <state_interface name="effort" />
+      </joint>
+      <joint name="rl_wheel_base_to_rl_wheel_joint">
+        <command_interface name="velocity" />
+        <state_interface name="position" />
+        <state_interface name="velocity" />
+        <state_interface name="effort" />
+      </joint>
+      <joint name="rr_wheel_base_to_rr_wheel_joint">
+        <command_interface name="velocity" />
+        <state_interface name="position" />
+        <state_interface name="velocity" />
+        <state_interface name="effort" />
+      </joint>
+    </ros2_control>
+    <!-- Load gazebo controller configuration -->
+    <xacro:if value="${use_sim}">
+      <xacro:gazebo.controller config_file="${controller_config_file}" namespace="${namespace}" />
+    </xacro:if>
   </xacro:macro>
 </robot>
