Commit message: Update controllers

File: urdf/common/imu.urdf.xacro (robot description, xacro)
@@ -1,4 +1,22 @@
 <?xml version="1.0" encoding="utf-8"?>
 <robot xmlns:xacro="http://wiki.ros.org/xacro">
+  <xacro:macro
+    name="imu_interface"
+    params="use_sim:=false
+            namespace:=''">
+    <xacro:property name="ns" value='${namespace + "/" if namespace else ""}' />
+    <sensor name="${ns}imu">
+      <state_interface name="orientation.x" />
+      <state_interface name="orientation.y" />
+      <state_interface name="orientation.z" />
+      <state_interface name="orientation.w" />
+      <state_interface name="angular_velocity.x" />
+      <state_interface name="angular_velocity.y" />
+      <state_interface name="angular_velocity.z" />
+      <state_interface name="linear_acceleration.x" />
+      <state_interface name="linear_acceleration.y" />
+      <state_interface name="linear_acceleration.z" />
+    </sensor>
+  </xacro:macro>
   <!-- Gauss noise macro -->
   <xacro:macro
@@ -24,4 +42,5 @@
             namespace:=''">
     <xacro:property name="ns" value='${namespace + "/" if namespace else ""}' />
+    <!-- Gazebo IMU -->
     <xacro:if value="${use_sim}">
       <gazebo reference="${reference_frame}">
@@ -65,6 +84,7 @@
       </gazebo>
     </xacro:if>
-    <xacro:unless value="${use_sim}">
-      <ros2_control name="${ns}imu" type="sensor">
+    <!-- ROS2 controller -->
+    <ros2_control name="${ns}imu" type="sensor">
+      <xacro:unless value="${use_sim}">
         <hardware>
           <!-- Hardware IMU sensor interface  -->
@@ -85,18 +105,6 @@
           <param name="world_frame">enu</param>
         </hardware>
-        <sensor name="${ns}imu">
-          <state_interface name="orientation.x" />
-          <state_interface name="orientation.y" />
-          <state_interface name="orientation.z" />
-          <state_interface name="orientation.w" />
-          <state_interface name="angular_velocity.x" />
-          <state_interface name="angular_velocity.y" />
-          <state_interface name="angular_velocity.z" />
-          <state_interface name="linear_acceleration.x" />
-          <state_interface name="linear_acceleration.y" />
-          <state_interface name="linear_acceleration.z" />
-        </sensor>
-      </ros2_control>
-    </xacro:unless>
+      </xacro:unless>
+    </ros2_control>
   </xacro:macro>
 </robot>

File: urdf/rover_a1.urdf.xacro (robot description, xacro)
@@ -2,12 +2,14 @@
 <robot name="rover_a1" xmlns:xacro="http://wiki.ros.org/xacro">
   <xacro:arg name="use_sim" default="false" />
-  <xacro:arg name="wheel_config_file"
-    default="$(find rover_description)/config/wheel_01.yaml" />
-  <xacro:arg name="controller_config_file"
-    default="$(find rover_controller)/config/wheel_01_controller.yaml" />
+  <xacro:arg name="imu_xyz" default="0.052 0.073 -0.006" />
+  <xacro:arg name="imu_rpy" default="0.0 0.0 -1.57" />
+  <xacro:arg name="wheel_config_file" default="$(find rover_description)/config/wheel_01.yaml" />
+  <xacro:arg name="controller_config_file" default="$(find rover_controller)/config/wheel_01_controller.yaml" />
   <xacro:arg name="namespace" default="" />
   <xacro:include filename="$(find rover_description)/urdf/rover_a1/rover_a1_macro.urdf.xacro" ns="rover" />
   <xacro:rover.rover_a1_robot
     use_sim="$(arg use_sim)"
+    imu_xyz="$(arg imu_xyz)"
+    imu_rpy="$(arg imu_rpy)"
     wheel_config_file="$(arg wheel_config_file)"
     controller_config_file="$(arg controller_config_file)"

File: urdf/rover_a1/rover_a1_macro.urdf.xacro (robot description, xacro)
@@ -9,11 +9,20 @@
             imu_rpy:='0.0 0.0 -1.57'
             namespace:=''">
+    <xacro:if value="${use_sim}">
+      <xacro:property name="imu_xyz" value="0.052 0.073 -0.006" />
+      <xacro:property name="imu_rpy" value="0.0 0.0 -1.57" />
+    </xacro:if>
     <xacro:property name="ns" value='${namespace + "/" if namespace else ""}' />
     <xacro:property name="wheel_config" value="${xacro.load_yaml(wheel_config_file)}" />
     <xacro:property name="wheelbase" value="0.2542" />
     <xacro:property name="wheel_mount_point_y" value="0.31301" />
+    <!-- Rover base macros -->
     <xacro:include filename="$(find rover_description)/urdf/rover_a1/base.urdf.xacro" ns="body" />
+    <!-- Rover wheel macros -->
     <xacro:include filename="$(find rover_description)/urdf/common/wheel.urdf.xacro" ns="wheel" />
+    <!-- IMU macros -->
     <xacro:include filename="$(find rover_description)/urdf/common/imu.urdf.xacro" ns="imu" />
+    <!-- Gazebo system macros -->
+    <xacro:include filename="$(find rover_description)/urdf/common/gazebo_system.urdf.xacro" ns="gazebo_system" />
     <!-- Rover body -->
     <xacro:body.body
@@ -47,4 +56,5 @@
     <!-- ROS2 Controller -->
     <ros2_control name="${ns}rover_system" type="system">
+      <!-- Joints -->
       <joint name="fl_wheel_base_to_fl_wheel_joint">
         <command_interface name="velocity" />
@@ -71,4 +81,7 @@
         <state_interface name="effort" />
       </joint>
+      <!-- IMU interfaces -->
+      <xacro:imu.imu_interface use_sim="${use_sim}" namespace="${namespace}" />
+      <!-- Hardware controller plugin -->
       <hardware>
         <xacro:if value="${use_sim}">
@@ -85,17 +98,6 @@
     <xacro:imu.imu use_sim="${use_sim}" reference_frame="imu_link" namespace="${namespace}" />
     <xacro:if value="${use_sim}">
-      <!-- Gazebo simulation system contorller plugin -->
-      <gazebo>
-        <plugin filename="gz_ros2_control-system" name="gz_ros2_control::GazeboSimROS2ControlPlugin">
-        <parameters>${controller_config_file}</parameters>
-          <ros>
-            <namespace>$(arg namespace)</namespace>
-            <remapping>drive_controller/cmd_vel:=cmd_vel</remapping>
-            <remapping>drive_controller/odom:=odometry/wheels</remapping>
-            <remapping>drive_controller/transition_event:=drive_controller/_transition_event</remapping>
-            <remapping>joint_state_broadcaster/transition_event:=joint_state_broadcaster/_transition_event</remapping>
-          </ros>
-        </plugin>
-      </gazebo>
+    <!-- Instantiate Gazebo System -->
+      <xacro:gazebo_system.controller controller_config_file="${controller_config_file}" namespace="${namespace}" />
     </xacro:if>
   </xacro:macro>
