Commit message: Add imu link and imu controller

File: urdf/rover_a1/base.urdf.xacro (robot description, xacro)
@@ -3,5 +3,7 @@
   <xacro:macro
     name="body"
-    params="wheel_radius">
+    params="wheel_radius
+            imu_xyz
+            imu_rpy">
     <link name="base_link" />
     <joint name="base_to_body_joint" type="fixed">
@@ -23,4 +25,10 @@
       </inertial>
     </link>
+    <joint name="body_to_imu_joint" type="fixed">
+      <origin xyz="${imu_xyz}" rpy="${imu_rpy}" />
+      <parent link="body_link" />
+      <child link="imu_link" />
+    </joint>
+    <link name="imu_link" />
     <joint name="body_to_footprint_joint" type="fixed">
       <origin xyz="0.0 0.0 -0.1359" rpy="0.0 0.0 0.0" />

File: urdf/rover_a1/rover_a1_macro.urdf.xacro (robot description, xacro)
@@ -6,4 +6,6 @@
             controller_config_file
             use_sim:=false
+            imu_xyz:='0.052 0.073 -0.006'
+            imu_rpy:='0.0 0.0 -1.57'
             namespace:=''">
     <xacro:property name="ns" value='${namespace + "/" if namespace else ""}' />
@@ -14,5 +16,7 @@
     <xacro:include filename="$(find rover_description)/urdf/common/wheel.urdf.xacro" ns="wheel" />
     <xacro:body.body
-      wheel_radius="${wheel_config['wheel_radius']}" />
+      wheel_radius="${wheel_config['wheel_radius']}"
+      imu_xyz="${imu_xyz}"
+      imu_rpy="${imu_rpy}" />
     <xacro:wheel.wheel
       config="${wheel_config}"
@@ -67,9 +71,43 @@
         </xacro:if>
         <xacro:unless value="${use_sim}">
-          <!-- Hardware interface system controller -->
-          <plugin>husarion_ugv_hardware_interfaces/RoverA1System</plugin>
+          <!-- Hardware controller system interface -->
+          <plugin>rover_hardware_interface/RoverA1System</plugin>
         </xacro:unless>
       </hardware>
     </ros2_control>
+    <xacro:unless value="${use_sim}">
+      <ros2_control name="${ns}imu" type="sensor">
+        <hardware>
+          <!-- Hardware IMU sensor interface  -->
+          <plugin>rover_hardware_interface/PhidgetImuSensor</plugin>
+          <param name="serial">-1</param>
+          <param name="hub_port">0</param>
+          <param name="data_interval_ms">8</param>
+          <param name="callback_delta_epsilon_ms">1</param>
+          <!-- Madgwick Filter Params -->
+          <param name="gain">0.00304</param>
+          <param name="zeta">0.00151</param>
+          <param name="mag_bias_x">0.0</param>
+          <param name="mag_bias_y">0.0</param>
+          <param name="mag_bias_z">0.0</param>
+          <param name="use_mag">true</param>
+          <param name="stateless">false</param>
+          <param name="remove_gravity_vector">false</param>
+          <param name="world_frame">enu</param>
+        </hardware>
+        <sensor name="${ns}imu">
+          <state_interface name="orientation.x" />
+          <state_interface name="orientation.y" />
+          <state_interface name="orientation.z" />
+          <state_interface name="orientation.w" />
+          <state_interface name="angular_velocity.x" />
+          <state_interface name="angular_velocity.y" />
+          <state_interface name="angular_velocity.z" />
+          <state_interface name="linear_acceleration.x" />
+          <state_interface name="linear_acceleration.y" />
+          <state_interface name="linear_acceleration.z" />
+        </sensor>
+      </ros2_control>
+    </xacro:unless>
     <xacro:if value="${use_sim}">
       <!-- Gazebo simulation system contorller plugin -->
